File: kicad_files/anubis.kicad_sch (KiCad schematic)
At the start: 234 parts, among them J1 A1001WR-S-04P, J2 A1001WR-S-04P, SW1 MX Switch, SW10 MX Switch, SW100 MX Switch, SW101 MX Switch, SW102 MX Switch, SW103 MX Switch, SW104 MX Switch, SW105 MX Switch, SW106 MX Switch, SW107 MX Switch, SW108 MX Switch, SW109 MX Switch, SW11 MX Switch, SW110 MX Switch, SW111 MX Switch, SW112 MX Switch, SW12 MX Switch, SW13 MX Switch, SW14 MX Switch, SW15 MX Switch, SW16 MX Switch, SW17 MX Switch, SW18 MX Switch, SW19 MX Switch, SW2 MX Switch, SW20 MX Switch, SW21 MX Switch, SW22 MX Switch, SW23 MX Switch, SW24 MX Switch, SW25 MX Switch, SW26 MX Switch, SW27 MX Switch, SW28 MX Switch, SW29 MX Switch, SW3 MX Switch, SW30 MX Switch, SW31 MX Switch, SW32 MX Switch, SW33 MX Switch, SW34 MX Switch, SW35 MX Switch, SW36 MX Switch, SW37 MX Switch, SW38 MX Switch, SW39 MX Switch, SW4 MX Switch, SW40 MX Switch, SW41 MX Switch, SW42 MX Switch, SW43 MX Switch, SW44 MX Switch, SW45 MX Switch, SW46 MX Switch, SW47 MX Switch, SW48 MX Switch, SW49 MX Switch, SW5 MX Switch, SW50 MX Switch, SW51 MX Switch, SW52 MX Switch, SW53 MX Switch, SW54 MX Switch, SW55 MX Switch, SW56 MX Switch, SW57 MX Switch, SW58 MX Switch, SW59 MX Switch, SW6 MX Switch, SW60 MX Switch, SW61 MX Switch, SW62 MX Switch, SW63 MX Switch, SW64 MX Switch, SW65 MX Switch, SW66 MX Switch, SW67 MX Switch, SW68 MX Switch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

Commit message: Remove F13, add screw points, move JST
- F13 layout removed: the old JST position was incompatible with F13 layout because it overlapped with the F1 key
- Screw points: added one for Idol and Ecliptica
- JST moved to the original WT80 position
Parts:
- removed D2: 1N4148W, acheron_Components:D_SOD-123, symbol Device:D
- removed R2, R4: 0R, Resistor_SMD:R_0805_2012Metric, symbol Device:R_Small
- removed SW18, SW19, SW2, SW20, SW21, SW22, SW23, SW24, SW25: MX Switch, acheron_MX_SolderMask:MX100, symbol acheronSymbols:Mechanical_Switch
Connections:
- net DL+ is gone; now on net D+: J2.3 (Pin_3)
- net DL- is gone; now on net D-: J2.2 (Pin_2)
- net C10: now also SW11.1; no longer SW11.2
- net C11: now also SW12.1; no longer SW12.2
- net C12: now also SW13.1; no longer SW13.2
- net at D11.2 (A): now also SW11.2; no longer SW11.1
- net at D12.2 (A): now also SW12.2; no longer SW12.1
- net at D13.2 (A): now also SW13.2; no longer SW13.1
Other:
- note added: "ANDROMEDA"
- note added: "WT80"
- moved on the sheet: SW11, SW12, SW13

Commit message: Some routing
Connections:
- net C0: no longer U2.38 (USART6_RX/TIM3_CH2/PC7)
- net C1: now also SW3.1; no longer U2.37 (I2S2_MCK/TIM3_CH1/USART6_TX/PC6)
- net C10: now also SW12.1; no longer SW11.1, U2.20 (PA4/USART2_CK)
- net C11: now also SW13.1; no longer SW12.1, U2.17 (PA3/TIM2_CH4/USART2_RX)
- net C12: now also SW14.1; no longer SW13.1, U2.16 (PA2/TIM2_CH3/USART2_TX)
- net C13: now also SW40.1; no longer SW14.1, U2.25 (PC5)
- net C14: no longer SW40.1, U2.43 (USART1_RX/TIM1_CH3/PA10)
- net C15: no longer U2.41 (USART1_CK/TIM1_CH1/PA8)
- net C16: no longer U2.40 (TIM3_CH4/I2S_CKIN/PC9)
- net C2: now also SW4.1; no longer SW3.1, U2.35 (SPI2_MISO/PB14)
- net C3: now also SW5.1; no longer SW4.1, U2.33 (PB12)
- net C4: now also SW6.1; no longer SW5.1, U2.29 (PB10/TIM2_CH3/SPI2_SCK/I2C2_SCL/I2S2_CK)
- net C5: now also SW7.1; no longer SW6.1, U2.27 (PB1/TIM3_CH4)
- net C6: now also SW8.1; no longer SW7.1, U2.24 (PC4)
- net C7: now also SW9.1; no longer SW8.1, U2.23 (PA7/SPI1_MOSI/TIM3_CH2)
- net C8: now also SW10.1; no longer SW9.1, U2.22 (PA6/TIM3_CH1/SPI1_MISO)
- net C9: now also SW11.1; no longer SW10.1, U2.21 (PA5/TIM2_CH1/SPI1_SCK)
- net E-PA0: no longer U2.14 (PA0/TIM2_CH1/USART2_CTS)
- net E-PB3: no longer U2.55 (JTDO-SWO/SPI1_SCK/SPI3_SCK/I2C2_SDA/TIM2_CH2/PB3)
- net E-PB4: no longer U2.56 (NJTRST/SPI1_MISO/SPI3_MISO/I2C3_SDA/TIM3_CH1/PB4)
- net E-PB5: no longer U2.57 (SPI1_MOSI/SPI3_MOSI/TIM3_CH2/PB5)
- net E-PB8: no longer U2.61 (I2C1_SCL/TIM4_CH3/TIM10_CH1/PB8)
- net E-PB9: no longer U2.62 (I2C1_SDA/TIM4_CH4/TIM11_CH1/PB9)
- net E-PC1: no longer U2.9 (PC1)
- net E-PC13: no longer U2.2 (PC13)
- net E-PC14: no longer U2.3 (PC14/OSC32_IN)
- net E-PC15: no longer U2.4 (PC15/OSC32_OUT)
- net E-PC2: no longer U2.10 (PC2/SPI2_MISO)
- net E-PC3: no longer U2.11 (PC3/SPI2_MOSI)
- net E-PD2: no longer U2.54 (PD2)
- net R0: now also D32.1 (K); no longer U2.52 (SPI3_MISO/PC11)
- net R1: now also D49.1 (K); no longer D32.1 (K), U2.53 (SPI3_MOSI/PC12)
- net R2: now also D66.1 (K), U2.27 (PB1/TIM3_CH4); no longer D49.1 (K), U2.51 (SPI3_SCK/I2S3_CK/PC10)
- net R3: no longer D66.1 (K), U2.50 (JTDI/TIM2_CH1/PA14)
- net R4: no longer U2.8 (PC0)
- net R5: no longer U2.15 (PA1/TIM2_CH2/USART2_RTS)
- no-connect marks 1 -> 0
Other:
- moved on the sheet: D10, D11, D12, D13, D14, D3, D32, D4, D49, D5, D6, D66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

Commit message: Some routing
Parts:
- added C1: 10u, Capacitor_SMD:C_0402_1005Metric, symbol Device:C_Small
- added C2: 100n, Capacitor_SMD:C_0402_1005Metric, symbol Device:C_Small
- added C3, C4: 1u, Capacitor_SMD:C_0805_2012Metric, symbol Device:C
- added C5: 10n, Capacitor_SMD:C_0402_1005Metric, symbol Device:C_Small
- added D1: 1N4148W, acheron_Components:D_SOD-123, symbol Device:D
- added D2: B5819W-SL, acheron_Components:D_SOD-123, symbol Device:D_Schottky
- added LED1, LED2: LED, acheron_Components:LED_THT_2.54mm, symbol acheron_Symbols:LED
- added Q1, Q2, Q4, Q5: 2N7002, Package_TO_SOT_SMD:SOT-23, symbol Transistor_FET:2N7002
- added Q3: AO3401A, Package_TO_SOT_SMD:SOT-23, symbol Transistor_FET:AO3401A
- added R1: 330k, Resistor_SMD:R_0402_1005Metric, symbol Device:R_Small
- added R10: 10k, Resistor_SMD:R_0805_2012Metric, symbol Device:R_Small
- added R15, R19, R22, R3, R9: 10k, Resistor_SMD:R_0402_1005Metric, symbol Device:R_Small
- added R17: 100, Resistor_SMD:R_0402_1005Metric, symbol Device:R_Small
- added R18, R21, R4, R5, R6: 100R, Resistor_SMD:R_0402_1005Metric, symbol Device:R_Small
- added R2: 1M, Resistor_SMD:R_0402_1005Metric, symbol Device:R_Small
- added R20: 1k, Resistor_SMD:R_0402_1005Metric, symbol Device:R_Small
- added R7, R8: 100k, Resistor_SMD:R_0805_2012Metric, symbol Device:R
- added SW1: K2-1187SQ-A4SW-06, acheron_Hardware:K2-1187SQ-A4SW-06, symbol Switch:SW_SPST
- added U1: SGM2007-3.3XN5/TR, acheron_Components:SOT-23-5, symbol acheron_Symbols:SGM2036
- renumbered C5 to C10, C6 to C11, C7 to C12, C8 to C13, C9 to C14, C10 to C15, C11 to C16, C12 to C17, C1 to C6, C2 to C7, C3 to C8, C4 to C9, D9 to D10, D10 to D11, D11 to D12, D12 to D13, D13 to D14, D14 to D15, D32 to D16, D15 to D17, D16 to D18, D17 to D19, D18 to D20, D19 to D21, D20 to D22, D21 to D23, D22 to D24, D23 to D25, D24 to D26, D25 to D27, D26 to D28, D27 to D29, D1 to D3, D28 to D30, D29 to D31, D30 to D32, D31 to D33, D49 to D34, D33 to D35, D34 to D36, D35 to D37, D36 to D38, D37 to D39, D3 to D4, D38 to D40, D39 to D41, D40 to D42, D41 to D43, D42 to D44, D43 to D45, D44 to D46, D45 to D47, D46 to D48, D47 to D49, D4 to D5, D48 to D50, D66 to D51, D50 to D52, D51 to D53, D52 to D54, D53 to D55, D54 to D56, D55 to D57, D56 to D58, D57 to D59, D5 to D6, D58 to D60, D59 to D61, D60 to D62, D61 to D63, D62 to D64, D63 to D65, D64 to D66, D65 to D67, D67 to D68, D68 to D69, D6 to D7, D69 to D70, D70 to D71, D71 to D72, D72 to D73, D73 to D74, D74 to D75, D75 to D76, D76 to D77, D77 to D78, D78 to D79, D7 to D8, D79 to D80, D80 to D81, D81 to D82, D82 to D83, D83 to D84, D84 to D85, D85 to D86, D86 to D87, D87 to D88, D88 to D89, D8 to D9, D89 to D90, D90 to D91, D91 to D92, D92 to D93, R1 to R11, R3 to R12, R5 to R13, R6 to R14, R7 to R16, SW108 to SW100, SW109 to SW101, SW110 to SW102, SW111 to SW103, SW112 to SW104, SW40 to SW15, SW15 to SW16, SW16 to SW17, SW17 to SW18, SW26 to SW19, SW1 to SW2, SW27 to SW20, SW28 to SW21, SW29 to SW22, SW30 to SW23, SW31 to SW24, SW32 to SW25, SW33 to SW26, SW34 to SW27, SW35 to SW28, SW36 to SW29, SW37 to SW30, SW38 to SW31, SW39 to SW32, SW58 to SW33, SW41 to SW34, SW42 to SW35, SW43 to SW36, SW44 to SW37, SW45 to SW38, SW46 to SW39, SW47 to SW40, SW48 to SW41, SW49 to SW42, SW50 to SW43, SW51 to SW44, SW52 to SW45, SW53 to SW46, SW54 to SW47, SW55 to SW48, SW56 to SW49, SW57 to SW50, SW75 to SW51, SW59 to SW52, SW60 to SW53, SW61 to SW54, SW62 to SW55, SW63 to SW56, SW64 to SW57, SW65 to SW58, SW66 to SW59, SW67 to SW60, SW68 to SW61, SW69 to SW62, SW70 to SW63, SW71 to SW64, SW72 to SW65, SW73 to SW66, SW74 to SW67, SW76 to SW68, SW77 to SW69, SW78 to SW70, SW79 to SW71, SW80 to SW72, SW81 to SW73, SW82 to SW74, SW83 to SW75, SW84 to SW76, SW85 to SW77, SW86 to SW78, SW87 to SW79, SW88 to SW80, SW89 to SW81, SW90 to SW82, SW91 to SW83, SW92 to SW84, SW93 to SW85, SW94 to SW86, SW95 to SW87, SW96 to SW88, SW97 to SW89, SW98 to SW90, SW99 to SW91, SW100 to SW92, SW101 to SW93, SW102 to SW94, SW103 to SW95, SW104 to SW96, SW105 to SW97, SW106 to SW98, SW107 to SW99, U1 to U2, U2 to U3
Connections:
- net 3V3: now also C4.1, D2.2 (A), R8.1, SW1.1 (A), U1.5 (OUT)
- net 5V: now also C3.1, D2.1 (K), Q3.2 (S), R15.2, R7.1, U1.1 (IN), U1.3 (EN)
- net BOOT0: now also C1.1, R1.1, R2.1, R3.2
- net C0: now also U3.39 (USART6_CK/TIM3_CH3/PC8)
- net C1: now also U3.38 (USART6_RX/TIM3_CH2/PC7)
- net C10: now also U3.22 (PA6/TIM3_CH1/SPI1_MISO)
- net C11: now also U3.21 (PA5/TIM2_CH1/SPI1_SCK)
- net C12: now also U3.20 (PA4/USART2_CK)
- net C13: now also U3.17 (PA3/TIM2_CH4/USART2_RX)
- net C2: now also U3.37 (I2S2_MCK/TIM3_CH1/USART6_TX/PC6)
- net C3: now also U3.35 (SPI2_MISO/PB14)
- net C4: now also U3.33 (PB12)
- net C5: now also U3.29 (PB10/TIM2_CH3/SPI2_SCK/I2C2_SCL/I2S2_CK)
- net C6: now also U3.26 (PB0/TIM3_CH3)
- net C7: now also U3.25 (PC5)
- net C8: now also U3.24 (PC4)
- net C9: now also U3.23 (PA7/SPI1_MOSI/TIM3_CH2)
- net CAPS_INDICATOR: now also U3.40 (TIM3_CH4/I2S_CKIN/PC9), R21.2; no longer U3.39 (USART6_CK/TIM3_CH3/PC8)
- net GND: now also C1.2, C2.2, C3.2, C4.2, C5.1, Q1.2 (S), Q2.2 (S), Q4.2 (S), Q5.2 (S), R10.2, R19.1, R2.2, R22.1, R7.2, R8.2, R9.1, U1.2 (GND)
- net LED_PWM: now also R18.2; no longer U3.26 (PB0/TIM3_CH3)
- net NRST: now also C2.1, R5.2
- net PB2/BOOT1: now also R10.1
- net R0: now also U3.41 (USART1_CK/TIM1_CH1/PA8)
- new net: D1.1 (K), R1.2
- new net: D1.2 (A), R6.2, SW1.2 (B)
- new net: Q2.3 (D), R4.1, R5.1
- new net: Q1.1 (G), R4.2
- new net: Q4.1 (G), R18.1, R19.2
- new net: Q4.3 (D), R15.1, R17.1
- new net: Q5.1 (G), R21.1, R22.2
- new net: Q1.3 (D), R3.1
- new net: LED1.K, LED2.K, R20.1
- new net: Q5.3 (D), R20.2
- new net: C5.2, U1.4 (BP/FB)
- new net: LED1.A, LED2.A, Q3.3 (D)
- new net: Q3.1 (G), R17.2
- new net: Q2.1 (G), R6.1, R9.2
Other:
- note added: "3V3"
- note added: "HARD RESET"

Commit message: Update submodules, more routing
Parts:
- removed Q1, Q2, Q5: 2N7002, Package_TO_SOT_SMD:SOT-23, symbol Transistor_FET:2N7002
- removed R10: 10k, Resistor_SMD:R_0805_2012Metric, symbol Device:R_Small
- removed R9: 10k, Resistor_SMD:R_0402_1005Metric, symbol Device:R_Small
- added LED3, LED4, LED5: LED, acheron_Components:LED_THT_2.54mm, symbol acheron_Symbols:LED
- added Q3, Q4, Q5, Q6: DTC123JKAT146, Package_TO_SOT_SMD:SOT-23, symbol acheron_Symbols:DTC123J
- added R20: 1k, Resistor_SMD:R_0402_1005Metric, symbol Device:R_Small
- added R7, R8: 10k, Resistor_SMD:R_0402_1005Metric, symbol Device:R_Small
- added U1: 2N7002DW, acheron_Components:SOT-363_SC-70-6, symbol acheron_Symbols:2N7002DW
- D1: Specification Small-signal switching diodes -> 400mW 1μA@75V 150mA SOD-123 small-signal witching diode
- R21: value 100R -> 1k; Manufacturer Part Number 0402WGF1000TCE -> 0402WGF1001TCE; Vendor Part Number LCSC C25076 -> LCSC C11702
- R22: value 10k -> 1k; Manufacturer Part Number 0402WGF1002TCE -> 0402WGF1001TCE; Vendor Part Number LCSC C25744 -> LCSC C11702
- renumbered Q3 to Q1, Q4 to Q2, R8 to R10, R20 to R23, R7 to R9, U1 to U2, U2 to U3, U3 to U4
Connections:
- net C14: now also U4.55 (JTDO-SWO/SPI1_SCK/SPI3_SCK/I2C2_SDA/TIM2_CH2/PB3)
- net C15: now also U4.54 (PD2)
- net C16: now also U4.53 (SPI3_MOSI/PC12)
- net CAPS_INDICATOR: now also Q3.1 (B); no longer R21.2
- net GND: now also U3.5 (SDA), U3.6 (SCL), Q3.2 (E), Q4.2 (E), Q5.2 (E), Q6.2 (E), R7.1, R8.2, U1.1 (S), U1.4 (S); no longer R22.1, U3.1 (A0), U3.2 (A1)
- net PB2/BOOT1: now also R8.1
- net SCL: now also U3.2 (A1); no longer U3.6 (SCL)
- net SDA: now also U3.1 (A0); no longer U3.5 (SDA)
- net at R4.1: now also U1.5 (G); no longer R5.1
- net at R4.2: now also R5.1, U1.6 (D)
- net at R22.2: now also Q6.3 (C); no longer R21.1
- net at R3.1: now also U1.3 (D)
- net at R23.2: now also Q3.3 (C)
- net INDICATOR1: now reaches U4.50 (JTDI/TIM2_CH1/PA14)
- net INDICATOR1: now also Q4.1 (B)
- net INDICATOR2: now reaches U4.51 (SPI3_SCK/I2S3_CK/PC10)
- net INDICATOR2: now also Q5.1 (B)
- net INDICATOR3: now reaches U4.52 (SPI3_MISO/PC11)
- net INDICATOR3: now also Q6.1 (B)
- net at LED1.A, LED2.A, Q1.3 (D): now also LED3.A, LED4.A, LED5.A
- net at R6.1: now also R7.2, U1.2 (G)
- new net: Q4.3 (C), R20.2
- new net: Q5.3 (C), R21.2
- new net: LED3.K, R20.1
- new net: LED4.K, R21.1
- new net: LED5.K, R22.1

Commit message: Finish routing and DRC, prepare for release
Parts:
- removed X2: Conn_01x02, acheron_Connectors:PinHeader_1x3_staggered_P2.54mm_Vertical, symbol Connector_Generic:Conn_01x03
- removed X3: EXTRA_PINS, acheron_Connectors:PinHeader_2x3_P2.54mm_Vertical, symbol Connector_Generic:Conn_02x03_Odd_Even
- added J3: Conn_01x06, acheron_Connectors:PinHeader_2x3_P2.54mm_Vertical, symbol Connector_Generic:Conn_02x03_Odd_Even
- added R8: 10k, Resistor_SMD:R_0402_1005Metric, symbol Device:R_Small
- SW69: footprint acheron_MX_SolderMask:MX_ISOEnter_Horizontal -> acheron_MX_SolderMask:MX_ISOEnter
- X2: renamed from X4; footprint acheron_Connectors:PinHeader_2x6_P2.54mm_Vertical -> acheron_Connectors:PinHeader_2x7_P2.54mm_Vertical; symbol Connector_Generic:Conn_02x06_Odd_Even -> Connector_Generic:Conn_02x07_Odd_Even
- renumbered C7 to C1, C1 to C2, C2 to C3, C3 to C4, C4 to C5, C5 to C6, C6 to C7, R15 to R1, R20 to R10, R21 to R11, R22 to R12, R23 to R13, R5 to R14, R6 to R15, R11 to R16, R12 to R17, R7 to R18, R9 to R19, R17 to R2, R10 to R20, R8 to R21, R13 to R22, R14 to R23, R16 to R24, R1 to R3, R18 to R4, R2 to R5, R19 to R6, R3 to R7, R4 to R9, U3 to U1, U1 to U2, U2 to U3
Connections:
- net E-PB3 is gone; now on net GND: X2.1 (Pin_1)
- net E-PB4 is gone; now on net E-PC15: X2.2 (Pin_2)
- net E-PD2 is gone; now on net E-PC0: X2.3 (Pin_3)
- net 3V3: now also X2.13 (Pin_13), J3.2 (Pin_2); no longer X2.9 (Pin_9)
- net 5V: now also X2.14 (Pin_14); no longer X2.11 (Pin_11)
- net C14: now also U4.56 (NJTRST/SPI1_MISO/SPI3_MISO/I2C3_SDA/TIM3_CH1/PB4); no longer U4.55 (JTDO-SWO/SPI1_SCK/SPI3_SCK/I2C2_SDA/TIM2_CH2/PB3)
- net C15: now also U4.55 (JTDO-SWO/SPI1_SCK/SPI3_SCK/I2C2_SDA/TIM2_CH2/PB3); no longer U4.54 (PD2)
- net C16: now also U4.54 (PD2); no longer U4.53 (SPI3_MOSI/PC12)
- net E-PA0: now also U4.14 (PA0/TIM2_CH1/USART2_CTS), X2.5 (Pin_5)
- net E-PB5: now also U4.57 (SPI1_MOSI/SPI3_MOSI/TIM3_CH2/PB5), J3.6 (Pin_6); no longer X2.4 (Pin_4)
- net E-PB8: now also U4.61 (I2C1_SCL/TIM4_CH3/TIM10_CH1/PB8), J3.5 (Pin_5); no longer X2.7 (Pin_7)
- net E-PB9: now also U4.62 (I2C1_SDA/TIM4_CH4/TIM11_CH1/PB9), J3.3 (Pin_3); no longer X2.12 (Pin_12)
- net E-PC13: now also U4.2 (PC13)
- net E-PC14: now also U4.3 (PC14/OSC32_IN), X2.4 (Pin_4); no longer X2.8 (Pin_8)
- net E-PC15: now also U4.4 (PC15/OSC32_OUT); no longer X2.10 (Pin_10)
- net E-PC2: now also U4.10 (PC2/SPI2_MISO), X2.11 (Pin_11)
- net E-PC3: now also U4.11 (PC3/SPI2_MOSI), X2.7 (Pin_7)
- net GND: now also U1.1 (A0), U1.2 (A1), X2.9 (Pin_9), J3.1 (Pin_1), R8.2; no longer U1.5 (SDA), U1.6 (SCL), X2.5 (Pin_5)
- net INDICATOR1: now also U4.51 (SPI3_SCK/I2S3_CK/PC10); no longer U4.50 (JTDI/TIM2_CH1/PA14)
- net INDICATOR2: now also U4.52 (SPI3_MISO/PC11); no longer U4.51 (SPI3_SCK/I2S3_CK/PC10)
- net INDICATOR3: now also U4.53 (SPI3_MOSI/PC12); no longer U4.52 (SPI3_MISO/PC11)
- net R1: now also U4.50 (JTDI/TIM2_CH1/PA14)
- net R3: now also U4.16 (PA2/TIM2_CH3/USART2_TX)
- net R4: now also U4.15 (PA1/TIM2_CH2/USART2_RTS)
- net R5: now also U4.9 (PC1)
- net SCL: now also U1.6 (SCL); no longer U1.2 (A1)
- net SDA: now also U1.5 (SDA); no longer U1.1 (A0)
- net XTAL_IN: now also C11.1; no longer C12.1
- net XTAL_OUT: now also C12.1; no longer C11.1
- net E-PB13: now reaches U4.34 (SPI2_SCK/I2S2_CK/PB13)
- net E-PB13: now also X2.10 (Pin_10)
- net E-PA10: now reaches U4.43 (USART1_RX/TIM1_CH3/PA10)
- net E-PA10: now also X2.8 (Pin_8)
- net E-PC0: now reaches U4.8 (PC0)
- net at LED1.A, LED2.A, LED3.A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: now also R8.1
- net PA9 renamed E-PA9
- net E-PA9: now also J3.4 (Pin_4)
- net RGB_3V3 renamed E-PB15
- net E-PB15: now also X2.12 (Pin_12)
Other:
- note added: "DB CONNS"
- note added: "GRAPHICS"
- note added: "INDICATORS"
- title: Noxary X60 -> Anubis PCB schematic
- moved on the sheet: C1, C10, C11, C12, C13, C14, C15, C16, C17, C2, C3, C4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
