File: kicad_files/anubis.kicad_sch (KiCad schematic)
At the start: 262 parts, among them J1 A1001WR-S-04P, J2 A1001WR-S-04P, Q1 AO3401A, Q2 2N7002, Q3 DTC123JKAT146, Q4 DTC123JKAT146, Q5 DTC123JKAT146, Q6 DTC123JKAT146, SW1 K2-1187SQ-A4SW-06, SW10 MX Switch, SW100 MX Switch, SW101 MX Switch, SW102 MX Switch, SW103 MX Switch, SW104 MX Switch, SW11 MX Switch, SW12 MX Switch, SW13 MX Switch, SW14 MX Switch, SW15 MX Switch, SW16 MX Switch, SW17 MX Switch, SW18 MX Switch, SW19 MX Switch, SW2 MX Switch, SW20 MX Switch, SW21 MX Switch, SW22 MX Switch, SW23 MX Switch, SW24 MX Switch, SW25 MX Switch, SW26 MX Switch, SW27 MX Switch, SW28 MX Switch, SW29 MX Switch, SW3 MX Switch, SW30 MX Switch, SW31 MX Switch, SW32 MX Switch, SW33 MX Switch, SW34 MX Switch, SW35 MX Switch, SW36 MX Switch, SW37 MX Switch, SW38 MX Switch, SW39 MX Switch, SW4 MX Switch, SW40 MX Switch, SW41 MX Switch, SW42 MX Switch, SW43 MX Switch, SW44 MX Switch, SW45 MX Switch, SW46 MX Switch, SW47 MX Switch, SW48 MX Switch, SW49 MX Switch, SW5 MX Switch, SW50 MX Switch, SW51 MX Switch, SW52 MX Switch, SW53 MX Switch, SW54 MX Switch, SW55 MX Switch, SW56 MX Switch, SW57 MX Switch, SW58 MX Switch, SW59 MX Switch, SW6 MX Switch, SW60 MX Switch, SW61 MX Switch, SW62 MX Switch, SW63 MX Switch, SW64 MX Switch, SW65 MX Switch, SW66 MX Switch, SW67 MX Switch, SW68 MX Switch, SW69 MX Switch, SW7 MX Switch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

Commit message: Metadata, QoL
Parts:
- X3: value Conn_01x06 -> EXTRA_PINS
Changed lines of the file:
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@@
   (title_block
     (title "Anubis PCB schematic")
-    (date "2022-05-21")
-    (rev "v1.0.3")
+    (date "2022-05-23")
+    (rev "v1.0.4")
     (company "Designed by Gondolindrim")
     (comment 1 "For the AcheronProject")
@@
     (in_bom no) (on_board yes)
     (property "Reference" "X3" (id 0) (at 782.955 376.555 0))
-    (property "Value" "Conn_01x06" (id 1) (at 782.955 379.095 0))
+    (property "Value" "EXTRA_PINS" (id 1) (at 782.955 379.095 0))
     (property "Footprint" "acheron_Connectors:PinHeader_2x3_P2.54mm_Vertical" (id 2) (at 781.685 385.445 0)
       (effects (font (size 1.27 1.27)) hide)
@@
     )
     (path "/3a146254-7ff6-44fa-bbbe-d41651ed1984"
-      (reference "X3") (unit 1) (value "Conn_01x06") (footprint "acheron_Connectors:PinHeader_2x3_P2.54mm_Vertical")
+      (reference "X3") (unit 1) (value "EXTRA_PINS") (footprint "acheron_Connectors:PinHeader_2x3_P2.54mm_Vertical")
     )
     (path "/4c975a56-2d4a-4f14-81bb-55c4a4e1277f"
